File: _autosave-K-75.kicad_pcb (KiCad board)
At the start: 2 copper layers, 314.3 x 123.8 mm, 177 parts, among them J1 Conn_01x04, SW1 SW_Push, U1 ATmega32U4-AU, Y1 Crystal_GND24_Small

Commit message: Tracing progress
Parts:
- C1, C2, C3, C4, C5, C6, C7, R1, R2, SW1: moved to B.Cu
- moved R2 518.3 mm to (341.5, 137.4), turned to 180 degrees
- moved SW1 507.0 mm to (349.4, 168.8), turned to 90 degrees
- moved C3 455.5 mm to (352.4, 147.9), turned to 90 degrees
- moved C1 437.0 mm to (339.0, 157.9), turned to 270 degrees
- moved C6 436.3 mm to (341.5, 139.6)
- moved C2 415.5 mm to (347.0, 157.9), turned to 90 degrees
- moved C7 394.5 mm to (354.5, 147.9), turned to 90 degrees
- moved R1 387.4 mm to (350.9, 156.6), turned to 90 degrees
- moved C5 385.9 mm to (332.4, 148.1), turned to 270 degrees
- moved C4 322.3 mm to (347.9, 139.7), turned to 180 degrees
- moved J1 49.9 mm to (348.9, 92.3), turned to 0 degrees
- moved Y1 7.62 mm to (342.9, 157.9), turned to 0 degrees
- moved U1 0.63 mm to (344.6, 148.0)
Connections:
- U1 pad 1: Net-(U1-Pad1) -> COL0
- U1 pad 10: COL2 -> ROW1
- U1 pad 11: COL3 -> ROW2
- U1 pad 12: COL7 -> ROW5
- U1 pad 18: COL10 -> ROW4
- U1 pad 19: COL11 -> ROW3
- U1 pad 20: COL12 -> Net-(U1-Pad20)
- U1 pad 21: COL13 -> Net-(U1-Pad21)
- U1 pad 26: Net-(U1-Pad26) -> COL13
- U1 pad 27: Net-(U1-Pad27) -> COL12
- U1 pad 28: COL4 -> COL11
- U1 pad 29: COL5 -> COL10
- U1 pad 30: COL6 -> COL9
- U1 pad 32: COL9 -> COL7
- U1 pad 36: ROW5 -> COL6
- U1 pad 37: ROW4 -> COL5
- U1 pad 38: ROW3 -> COL4
- U1 pad 39: ROW2 -> COL3
- U1 pad 40: ROW1 -> COL2
- U1 pad 41: ROW0 -> COL1
- U1 pad 8: COL0 -> Net-(U1-Pad8)
- U1 pad 9: COL1 -> ROW0
Routing:
- net GND: track 0.00 -> 69.3 mm
- net COL0: track 405.3 -> 457.7 mm
- net +5V: track 0.00 -> 51.9 mm, vias 0 -> 3
- net COL10: track 199.6 -> 250.4 mm
- net COL9: track 246.2 -> 296.5 mm
- net COL8: track 262.4 -> 312.1 mm
- net COL7: track 255.1 -> 304.3 mm
- net COL1: track 399.6 -> 448.3 mm
- net COL2: track 374.2 -> 422.1 mm
- net COL3: track 331.0 -> 378.4 mm
- net COL4: track 311.1 -> 358.1 mm
- net COL5: track 316.8 -> 363.4 mm
- net COL6: track 273.9 -> 320.1 mm
- net ROW1: track 257.2 -> 295.3 mm, vias 0 -> 2
- net ROW2: track 257.2 -> 290.4 mm, vias 0 -> 2
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