File: K-75.kicad_pcb (KiCad board)
At the start: 2 copper layers, 177 parts, among them J1 Conn_01x04, SW1 SW_Push, U1 ATmega32U4-AU, Y1 Crystal_GND24_Small

Commit message: Key placement
Parts:
- moved K_upArrow1 569.6 mm to (338.2, 169.9)
- moved K_rightShift1 563.4 mm to (307.3, 165.2)
- moved K_leftAlt1 392.9 mm to (116.7, 184.3)
- moved K_Win1 392.8 mm to (92.8, 184.3)
- moved K_N1 388.6 mm to (204.9, 165.2)
- moved K_capsLock1 363.7 mm to (73.9, 146.2)
- moved K_J1 359.0 mm to (214.4, 146.2)
- moved K_R1 343.1 mm to (152.4, 127.1)
- moved K_Z1 340.2 mm to (109.6, 165.2)
- moved K_;1 320.2 mm to (271.5, 146.2)
- moved K_F7 312.6 mm to (209.6, 84.2)
- moved K_,1 309.9 mm to (243.0, 165.2)
- moved K_9 290.5 mm to (238.1, 108.1)
- moved K_5 223.9 mm to (161.9, 108.1)
- moved K_2 193.6 mm to (104.8, 108.1)
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Changed lines of the file:
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@@
   )
   (module MX_Only:MXOnly-1U-Hotswap (layer F.Cu)
-    (at -182.051 -9.976)
+    (at 109.601 165.227)
     (attr smd)
     (fp_text reference K_Z1 (at 0 3.175) (layer F.Fab)
@@
       (rotate (xyz 0 0 0))
     )
+    (model ${KIPRJMOD}/MX_Alps_Hybrid/MX_Only.pretty/3d_shapes/CPG151101S11.wrl
+      (offset (xyz 0 0 -1.75))
+      (scale (xyz 0.4 0.4 0.4))
+      (rotate (xyz 0 0 0))
+    )
   )
   (module MX_Only:MXOnly-1U-Hotswap (layer F.Cu)
@@
   )
   (module MX_Only:MXOnly-1.25U-Hotswap (layer F.Cu)
-    (at -259.30975 10.224)
+    (at 92.837 184.277)
     (attr smd)
     (fp_text reference K_Win1 (at 0 3.048) (layer F.Fab)
@@
       (rotate (xyz 0 0 0))
     )
+    (model ${KIPRJMOD}/MX_Alps_Hybrid/MX_Only.pretty/3d_shapes/CPG151101S11.wrl
+      (offset (xyz 0 0 -1.75))
+      (scale (xyz 0.4 0.4 0.4))
+      (rotate (xyz 0 0 0))
+    )
   )
   (module MX_Only:MXOnly-1U-Hotswap (layer F.Cu)
@@
   )
   (module MX_Only:MXOnly-1U-Hotswap (layer F.Cu)
-    (at -202.251 -9.976)
+    (at 338.201 169.926)
     (attr smd)
     (fp_text reference K_upArrow1 (at 0 3.175) (layer F.Fab)
@@
       (rotate (xyz 0 0 0))
     )
+    (model ${KIPRJMOD}/MX_Alps_Hybrid/MX_Only.pretty/3d_shapes/CPG151101S11.wrl
+      (offset (xyz 0 0 -1.75))
+      (scale (xyz 0.4 0.4 0.4))
+      (rotate (xyz 0 0 0))
+    )
   )
   (module MX_Only:MXOnly-1U-Hotswap (layer F.Cu)
@@
   )
   (module MX_Only:MXOnly-1.25U-Hotswap (layer F.Cu)
-    (at -234.34975 10.224)
+    (at 307.34 165.227)
     (attr smd)
     (fp_text reference K_rightShift1 (at 0 3.048) (layer F.Fab)
@@
   )
   (module MX_Only:MXOnly-1U-Hotswap (layer F.Cu)
-    (at -161.851 -10.616)
+    (at 152.4 127.127)
     (attr smd)
     (fp_text reference K_R1 (at 0 3.175) (layer F.Fab)
@@
       (rotate (xyz 0 0 0))
     )
+    (model ${KIPRJMOD}/MX_Alps_Hybrid/MX_Only.pretty/3d_shapes/CPG151101S11.wrl
+      (offset (xyz 0 0 -1.75))
+      (scale (xyz 0.4 0.4 0.4))
+      (rotate (xyz 0 0 0))
+    )
   )
   (module MX_Only:MXOnly-1U-Hotswap (layer F.Cu)
@@
   )
   (module MX_Only:MXOnly-1U-Hotswap (layer F.Cu)
-    (at -141.651 -10.616)
+    (at 204.851 165.227)
     (attr smd)
     (fp_text reference K_N1 (at 0 3.175) (layer F.Fab)
@@
       (rotate (xyz 0 0 0))
     )
+    (model ${KIPRJMOD}/MX_Alps_Hybrid/MX_Only.pretty/3d_shapes/CPG151101S11.wrl
+      (offset (xyz 0 0 -1.75))
+      (scale (xyz 0.4 0.4 0.4))
+      (rotate (xyz 0 0 0))
+    )
   )
   (module MX_Only:MXOnly-1U-Hotswap (layer F.Cu)
@@
   )
   (module MX_Only:MXOnly-1.25U-Hotswap (layer F.Cu)
-    (at -224.82975 -9.976)
+    (at 116.713 184.277)
     (attr smd)
     (fp_text reference K_leftAlt1 (at 0 3.048) (layer F.Fab)
@@
       (rotate (xyz 0 0 0))
     )
+    (model ${KIPRJMOD}/MX_Alps_Hybrid/MX_Only.pretty/3d_shapes/CPG151101S11.wrl
+      (offset (xyz 0 0 -1.75))
+      (scale (xyz 0.4 0.4 0.4))
+      (rotate (xyz 0 0 0))
+    )
   )
   (module MX_Only:MXOnly-1U-Hotswap (layer F.Cu)
@@
   )
   (module MX_Only:MXOnly-1U-Hotswap (layer F.Cu)
-    (at -108.311 -11.256)
+    (at 214.376 146.177)
     (attr smd)
     (fp_text reference K_J1 (at 0 3.175) (layer F.Fab)
@@
       (rotate (xyz 0 0 0))
     )
+    (model ${KIPRJMOD}/MX_Alps_Hybrid/MX_Only.pretty/3d_shapes/CPG151101S11.wrl
+      (offset (xyz 0 0 -1.75))
+      (scale (xyz 0.4 0.4 0.4))
+      (rotate (xyz 0 0 0))
+    )
   )
   (module MX_Only:MXOnly-1U-Hotswap (layer F.Cu)
@@
   )
   (module MX_Only:MXOnly-1U-Hotswap (layer F.Cu)
-    (at -88.111 -11.256)
+    (at 209.55 84.201)
     (attr smd)
     (fp_text reference K_F7 (at 0 3.175) (layer F.Fab)
@@
       (rotate (xyz 0 0 0))
     )
+    (model ${KIPRJMOD}/MX_Alps_Hybrid/MX_Only.pretty/3d_shapes/CPG151101S11.wrl
+      (offset (xyz 0 0 -1.75))
+      (scale (xyz 0.4 0.4 0.4))
+      (rotate (xyz 0 0 0))
+    )
   )
   (module MX_Only:MXOnly-1U-Hotswap (layer F.Cu)
@@
   )
   (module MX_Only:MXOnly-1U-Hotswap (layer F.Cu)
-    (at -67.911 -11.256)
+    (at 66.675 84.201)
     (attr smd)
     (fp_text reference K_Esc1 (at 0 3.175) (layer F.Fab)
@@
       (rotate (xyz 0 0 0))
     )
+    (model ${KIPRJMOD}/MX_Alps_Hybrid/MX_Only.pretty/3d_shapes/CPG151101S11.wrl
+      (offset (xyz 0 0 -1.75))
+      (scale (xyz 0.4 0.4 0.4))
+      (rotate (xyz 0 0 0))
+    )
   )
   (module MX_Only:MXOnly-2.25U-Hotswap (layer F.Cu)
@@
   )
   (module MX_Only:MXOnly-1.75U-Hotswap (layer F.Cu)
-    (at -254.54725 -9.976)
+    (at 73.914 146.177)
     (attr smd)
     (fp_text reference K_capsLock1 (at 0 3.175) (layer F.Fab)
@@
       (rotate (xyz 0 0 0))
     )
+    (model ${KIPRJMOD}/MX_Alps_Hybrid/MX_Only.pretty/3d_shapes/CPG151101S11.wrl
+      (offset (xyz 0 0 -1.75))
+      (scale (xyz 0.4 0.4 0.4))
+      (rotate (xyz 0 0 0))
+    )
   )
   (module MX_Only:MXOnly-1U-Hotswap (layer F.Cu)
@@
   )
   (module MX_Only:MXOnly-1U-Hotswap (layer F.Cu)
-    (at -7.311 -11.256)
+    (at 271.526 146.177)
     (attr smd)
     (fp_text reference K_;1 (at 0 3.175) (layer F.Fab)
@@
       (rotate (xyz 0 0 0))
     )
+    (model ${KIPRJMOD}/MX_Alps_Hybrid/MX_Only.pretty/3d_shapes/CPG151101S11.wrl
+      (offset (xyz 0 0 -1.75))
+      (scale (xyz 0.4 0.4 0.4))
+      (rotate (xyz 0 0 0))
+    )
   )
   (module MX_Only:MXOnly-1U-Hotswap (layer F.Cu)
@@
   )
   (module MX_Only:MXOnly-1U-Hotswap (layer F.Cu)
-    (at -16.671 -31.456)
+    (at 238.125 108.077)
     (attr smd)
     (fp_text reference K_9 (at 0 3.175) (layer F.Fab)
@@
       (rotate (xyz 0 0 0))
     )
+    (model ${KIPRJMOD}/MX_Alps_Hybrid/MX_Only.pretty/3d_shapes/CPG151101S11.wrl
+      (offset (xyz 0 0 -1.75))
+      (scale (xyz 0.4 0.4 0.4))
+      (rotate (xyz 0 0 0))
+    )
   )
   (module MX_Only:MXOnly-1U-Hotswap (layer F.Cu)
@@
   )
   (module MX_Only:MXOnly-1U-Hotswap (layer F.Cu)
-    (at -27.511 -11.256)
+    (at 161.925 108.077)
     (attr smd)
     (fp_text reference K_5 (at 0 3.175) (layer F.Fab)
@@
       (rotate (xyz 0 0 0))
     )
+    (model ${KIPRJMOD}/MX_Alps_Hybrid/MX_Only.pretty/3d_shapes/CPG151101S11.wrl
+      (offset (xyz 0 0 -1.75))
+      (scale (xyz 0.4 0.4 0.4))
+      (rotate (xyz 0 0 0))
+    )
   )
   (module MX_Only:MXOnly-1U-Hotswap (layer F.Cu)
@@
   )
   (module MX_Only:MXOnly-1U-Hotswap (layer F.Cu)
-    (at -47.711 -11.256)
+    (at 104.775 108.077)
     (attr smd)
     (fp_text reference K_2 (at 0 3.175) (layer F.Fab)
@@
       (rotate (xyz 0 0 0))
     )
+    (model ${KIPRJMOD}/MX_Alps_Hybrid/MX_Only.pretty/3d_shapes/CPG151101S11.wrl
+      (offset (xyz 0 0 -1.75))
+      (scale (xyz 0.4 0.4 0.4))
+      (rotate (xyz 0 0 0))
+    )
   )
   (module MX_Only:MXOnly-1U-Hotswap (layer F.Cu)
@@
   )
   (module MX_Only:MXOnly-1U-Hotswap (layer F.Cu)
-    (at 3.529 -31.456)
+    (at 242.951 165.227)
     (attr smd)
     (fp_text reference K_,1 (at 0 3.175) (layer F.Fab)
@@
       (rotate (xyz 0 0 0))
     )
+    (model ${KIPRJMOD}/MX_Alps_Hybrid/MX_Only.pretty/3d_shapes/CPG151101S11.wrl
+      (offset (xyz 0 0 -1.75))
+      (scale (xyz 0.4 0.4 0.4))
+      (rotate (xyz 0 0 0))
+    )

Commit message: Finished key placement with 3d models
Parts:
- K_rightShift1: footprint MX_Only:MXOnly-1.25U-Hotswap -> MX_Only:MXOnly-1.75U-Hotswap
- moved K_pgUp1 624.7 mm to (361.9, 127.1)
- moved K_rightArrow1 558.0 mm to (357.3, 189.0)
- moved K_]1 531.6 mm to (304.8, 127.1)
- moved K_\1 531.0 mm to (328.7, 127.1)
- moved K_leftArrow1 520.0 mm to (319.2, 189.0)
- moved K_home1 519.1 mm to (361.9, 108.1)
- moved K_end1 511.4 mm to (361.9, 165.2)
- moved K_P1 509.5 mm to (266.7, 127.1)
- moved K_downArrow1 508.4 mm to (338.2, 189.0)
- moved K_Fn1 506.2 mm to (276.2, 184.3)
- moved K_O1 472.3 mm to (247.7, 127.1)
- moved K_U1 456.6 mm to (209.6, 127.1)
- moved K_F11 452.5 mm to (290.6, 84.2)
- moved K_G1 444.4 mm to (176.3, 146.2)
- moved K_M1 440.2 mm to (223.9, 165.2)
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
Commit message: Finished diode placement
Parts:
- D1, D10, D11, D12, D13, D14, D15, D16, D17, D18, D19, D2, D20, D21, D22, D23, D24, D25, D26, D27, D28, D29, D3, D30, D31, D32, D33, D34, D35, D36, D37, D38, D39, D4, D40, D41, D42, D43, D44, D45, D46, D47, D48, D49, D5, D50, D51, D52, D53, D54, D55, D56, D57, D59, D6, D60, D61, D62, D63, D64, D65, D66, D67, D68, D69, D7, D70, D71, D72, D73, D74, D75, D76, D77, D78, D79, D8, D80, D81, D82, D83, D9: footprint Diode_SMD:D_SOD-323 -> Diode_SMD:D_SOD-123; moved to B.Cu
- moved D73 528.0 mm to (367.0, 169.3), turned to 90 degrees
- moved D72 525.5 mm to (343.3, 174.0), turned to 90 degrees
- moved D81 496.9 mm to (324.2, 193.0), turned to 90 degrees
- moved D44 477.4 mm to (367.0, 131.2), turned to 90 degrees
- moved D80 469.5 mm to (300.4, 188.3), turned to 90 degrees
- moved D71 469.0 mm to (312.3, 169.3), turned to 90 degrees
- moved D79 458.9 mm to (281.3, 188.3), turned to 90 degrees
- moved D70 451.6 mm to (286.1, 169.3), turned to 90 degrees
- moved D83 450.7 mm to (362.3, 193.0), turned to 90 degrees
- moved D43 440.1 mm to (333.8, 131.2), turned to 90 degrees
- moved D78 438.3 mm to (262.4, 188.3), turned to 90 degrees
- moved D14 438.0 mm to (338.5, 88.3), turned to 90 degrees
- moved D69 430.2 mm to (267.1, 169.3), turned to 90 degrees
- moved D42 420.3 mm to (309.9, 131.2), turned to 90 degrees
- moved D68 409.1 mm to (248.0, 169.3), turned to 90 degrees
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
Commit message: Edge cuts
Parts:
- U1: moved to B.Cu
- moved U1 419.0 mm to (343.9, 148.0)
Other:
- board outline added: 314.3 x 123.8 mm

Commit message: Finished diode matrix
Routing:
- net ROW5: track 0.00 -> 290.1 mm
- net ROW4: track 0.00 -> 287.6 mm
- net ROW0: track 0.00 -> 266.7 mm
- net ROW2: track 0.00 -> 257.2 mm
- net ROW1: track 0.00 -> 257.2 mm
- net ROW3: track 0.00 -> 247.7 mm
- net Net-(D13-Pad2): track 0.00 -> 9.30 mm
- net Net-(D10-Pad2): track 0.00 -> 9.30 mm
- net Net-(D74-Pad2): track 0.00 -> 9.19 mm
- net Net-(D72-Pad2): track 0.00 -> 9.18 mm
- net Net-(D6-Pad2): track 0.00 -> 9.18 mm
- net Net-(D32-Pad2): track 0.00 -> 8.95 mm
- net Net-(D44-Pad2): track 0.00 -> 8.95 mm
- net Net-(D40-Pad2): track 0.00 -> 8.95 mm
- net Net-(D80-Pad2): track 0.00 -> 8.89 mm
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
Commit message: Finished vertical matrix trace routing
Parts:
- moved D63 19.2 mm to (152.9, 169.3)
- moved D62 19.1 mm to (133.7, 169.3)
- moved K_C1 19.0 mm to (147.7, 165.2)
- moved K_X1 19.0 mm to (128.7, 165.2)
Routing:
- net COL11: track 0.00 -> 134.2 mm, vias 0 -> 6
- net COL9: track 0.00 -> 133.2 mm, vias 0 -> 6
- net COL8: track 0.00 -> 129.9 mm, vias 0 -> 6
- net COL12: track 0.00 -> 129.6 mm, vias 0 -> 5
- net COL1: track 2.49 -> 131.8 mm, vias 1 -> 6
- net COL5: track 0.00 -> 126.0 mm, vias 0 -> 6
- net COL2: track 0.00 -> 124.9 mm, vias 0 -> 6
- net COL13: track 0.00 -> 124.5 mm, vias 0 -> 5
- net COL0: track 0.00 -> 118.0 mm, vias 0 -> 6
- net COL10: track 0.00 -> 106.2 mm, vias 0 -> 5
- net COL6: track 0.00 -> 103.3 mm, vias 0 -> 5
- net COL7: track 0.00 -> 103.1 mm, vias 0 -> 5
- net COL3: track 0.00 -> 101.2 mm, vias 0 -> 5
- net COL4: track 0.00 -> 100.8 mm, vias 0 -> 5
- net COL14: track 0.00 -> 89.1 mm, vias 0 -> 5

Commit message: Tracing progress
Parts:
- C1, C2, C3, C4, C5, C6, C7, J1, R1, R2, SW1, Y1: moved to B.Cu
- moved R2 518.3 mm to (341.5, 137.4), turned to 180 degrees
- moved SW1 507.0 mm to (349.4, 168.8), turned to 90 degrees
- moved Y1 494.6 mm to (342.8, 159.9)
- moved J1 478.9 mm to (348.9, 92.3)
- moved C3 455.5 mm to (352.4, 147.9), turned to 90 degrees
- moved C1 437.2 mm to (338.7, 160.4), turned to 270 degrees
- moved C6 436.3 mm to (341.5, 139.6)
- moved C2 416.7 mm to (347.6, 159.9), turned to 90 degrees
- moved C7 394.5 mm to (354.5, 147.9), turned to 90 degrees
- moved R1 387.4 mm to (350.9, 156.6), turned to 90 degrees
- moved C5 385.9 mm to (332.4, 148.1), turned to 270 degrees
- moved C4 322.3 mm to (347.9, 139.7), turned to 180 degrees
- moved U1 0.63 mm to (344.6, 148.0), turned to 180 degrees
Connections:
- U1 pad 1: Net-(U1-Pad1) -> COL0
- U1 pad 10: Net-(U1-Pad10) -> ROW1
- U1 pad 11: Net-(U1-Pad11) -> ROW2
- U1 pad 12: Net-(U1-Pad12) -> ROW5
- U1 pad 18: Net-(U1-Pad18) -> ROW4
- U1 pad 19: Net-(U1-Pad19) -> ROW3
- U1 pad 25: Net-(U1-Pad25) -> COL14
- U1 pad 26: Net-(U1-Pad26) -> COL13
- U1 pad 27: Net-(U1-Pad27) -> COL12
- U1 pad 28: Net-(U1-Pad28) -> COL11
- U1 pad 29: Net-(U1-Pad29) -> COL10
- U1 pad 30: Net-(U1-Pad30) -> COL9
- U1 pad 31: Net-(U1-Pad31) -> COL8
- U1 pad 32: Net-(U1-Pad32) -> COL7
- U1 pad 36: Net-(U1-Pad36) -> COL6
- U1 pad 37: Net-(U1-Pad37) -> COL5
- U1 pad 38: Net-(U1-Pad38) -> COL4
- U1 pad 39: Net-(U1-Pad39) -> COL3
- U1 pad 40: Net-(U1-Pad40) -> COL2
- U1 pad 41: Net-(U1-Pad41) -> COL1
- U1 pad 9: Net-(U1-Pad9) -> ROW0
Routing:
- net COL0: track 118.0 -> 457.7 mm
- net COL1: track 131.8 -> 448.3 mm
- net COL2: track 124.9 -> 422.1 mm
- net COL3: track 101.2 -> 378.4 mm
- net COL4: track 100.8 -> 358.1 mm
- net COL5: track 126.0 -> 363.4 mm
- net COL6: track 103.3 -> 320.1 mm
- net COL7: track 103.1 -> 304.3 mm
- net COL8: track 129.9 -> 312.1 mm
- net COL9: track 133.2 -> 296.5 mm
- net COL10: track 106.2 -> 250.4 mm
- net COL11: track 134.2 -> 259.4 mm
- net COL12: track 129.6 -> 235.0 mm
- net COL13: track 124.5 -> 206.2 mm
- net +5V: track 0.00 -> 51.9 mm, vias 0 -> 3
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
Commit message: Improved routing
Parts:
- moved C1 2.53 mm to (339.0, 157.9)
- moved C2 2.10 mm to (347.0, 157.9)
- moved C5 2.08 mm to (333.2, 150.0), turned to 180 degrees
- moved Y1 2.04 mm to (342.9, 157.9)
Connections:
- U1 pad 1: COL0 -> ROW0
- U1 pad 25: COL14 -> COL13
- U1 pad 26: COL13 -> COL12
- U1 pad 27: COL12 -> COL11
- U1 pad 28: COL11 -> COL10
- U1 pad 29: COL10 -> COL9
- U1 pad 30: COL9 -> COL8
- U1 pad 31: COL8 -> COL7
- U1 pad 32: COL7 -> COL6
- U1 pad 36: COL6 -> COL5
- U1 pad 37: COL5 -> COL4
- U1 pad 38: COL4 -> COL3
- U1 pad 39: COL3 -> COL2
- U1 pad 40: COL2 -> COL1
- U1 pad 41: COL1 -> COL0
- U1 pad 8: Net-(U1-Pad8) -> COL14
- U1 pad 9: ROW0 -> Net-(U1-Pad9)
Routing:
- net ROW0: track 266.7 -> 325.6 mm
- net ROW1: track 257.2 -> 295.3 mm, vias 0 -> 2
- net ROW2: track 257.2 -> 290.4 mm, vias 0 -> 2
- net GND: track 50.5 -> 76.5 mm
- net Net-(C2-Pad1): track 0.00 -> 8.73 mm
- net Net-(C1-Pad1): track 0.00 -> 7.60 mm
- net COL12: track 235.0 -> 240.5 mm
- net +5V: track 51.9 -> 57.2 mm
- net COL6: track 320.1 -> 323.8 mm
- net COL0: track 457.7 -> 454.4 mm
- net COL13: track 206.2 -> 207.7 mm
- net COL7: track 304.3 -> 305.5 mm
- net COL11: track 259.4 -> 260.6 mm
- net COL8: track 312.1 -> 313.3 mm
- net COL10: track 250.4 -> 251.6 mm
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