File: K-75.sch (KiCad schematic (older format))
At the start: 193 parts, among them J1 Conn_01x04, SW1 SW_Push, U1 ATmega32U4-AU, Y1 Crystal_GND24_Small

Commit message: Finished routing
Connections:
- net COL14: now also U1.12 (PB7); no longer U1.10 (PB2)
- net RGBLED: now also U1.10 (PB2); no longer U1.20 (PD2)
- net ROW3: now also D59.1 (K), U1.11 (PB3); no longer U1.19 (PD1)
- net ROW4: now also U1.22 (PD5); no longer U1.18 (PD0)
- net ROW5: now also U1.21 (PD3); no longer U1.12 (PB7)
Changed lines of the file:
@@
 Text GLabel 4750 9850 2    50   Input ~ 0
 COL2
-Text GLabel 4750 9950 2    50   Input ~ 0
-COL3
 Text GLabel 4750 10050 2    50   Input ~ 0
 COL4
@@
 Text GLabel 4750 9050 2    50   Input ~ 0
 COL12
-Text GLabel 4750 8850 2    50   Input ~ 0
-COL13
-Text GLabel 4750 7450 2    50   Input ~ 0
-COL14
 Text GLabel 4750 9450 2    50   Input ~ 0
 ROW0
@@
 Text GLabel 4750 7350 2    50   Input ~ 0
 ROW2
-Text GLabel 4750 8550 2    50   Input ~ 0
+Text GLabel 4750 7550 2    50   Input ~ 0
 ROW3
-Text GLabel 4750 8450 2    50   Input ~ 0
+Text GLabel 4750 8950 2    50   Input ~ 0
 ROW4
-Text GLabel 4750 7950 2    50   Input ~ 0
+Text GLabel 4750 8750 2    50   Input ~ 0
 ROW5
-Text GLabel 4750 8650 2    50   Input ~ 0
-RGBLED
 $Comp
 L LED:WS2812B D58
@@
 $EndComp
 Connection ~ 10550 8000
+Text GLabel 4750 8850 2    50   Input ~ 0
+COL13
+Text GLabel 4750 7450 2    50   Input ~ 0
+RGBLED
+Wire Wire Line
+	10000 4550 11450 4550
+Connection ~ 10000 4550
+Text GLabel 4750 9950 2    50   Input ~ 0
+COL3
+Text GLabel 4750 7950 2    50   Input ~ 0
+COL14
 $EndSCHEMATC

Commit message: Added USB traces
Connections:
- net VCC is gone; now on net +5V: J1.4 (Pin_4)
Changed lines of the file:
@@
 Wire Wire Line
 	6100 10800 5900 10800
-$Comp
-L power:VCC #PWR0112
-U 1 1 62554D45
-P 5900 10800
-F 0 "#PWR0112" H 5900 10650 50  0001 C CNN
-F 1 "VCC" H 5917 10973 50  0000 C CNN
-F 2 "" H 5900 10800 50  0001 C CNN
-F 3 "" H 5900 10800 50  0001 C CNN
-	1    5900 10800
-	1    0    0    -1
-$EndComp
 Wire Wire Line
 	10900 3250 10900 5000
@@
 Text GLabel 4750 7950 2    50   Input ~ 0
 COL14
+$Comp
+L power:+5V #PWR?
+U 1 1 62738D63
+P 5900 10800
+F 0 "#PWR?" H 5900 10650 50  0001 C CNN
+F 1 "+5V" H 5915 10973 50  0000 C CNN
+F 2 "" H 5900 10800 50  0001 C CNN
+F 3 "" H 5900 10800 50  0001 C CNN
+	1    5900 10800
+	1    0    0    -1
+$EndComp
 $EndSCHEMATC

Commit message: Finished traces
Connections:
- net rotarySwitch: now reaches U1.18 (PD0)
- net A: now reaches U1.19 (PD1)
- net B: now reaches U1.20 (PD2)
Changed lines of the file:
@@
 COL14
 $Comp
-L power:+5V #PWR?
+L power:+5V #PWR0112
 U 1 1 62738D63
 P 5900 10800
-F 0 "#PWR?" H 5900 10650 50  0001 C CNN
+F 0 "#PWR0112" H 5900 10650 50  0001 C CNN
 F 1 "+5V" H 5915 10973 50  0000 C CNN
 F 2 "" H 5900 10800 50  0001 C CNN
@@
 	1    0    0    -1
 $EndComp
+Text GLabel 4750 8450 2    50   Input ~ 0
+rotarySwitch
+Text GLabel 4750 8550 2    50   Input ~ 0
+A
+Text GLabel 4750 8650 2    50   Input ~ 0
+B
 $EndSCHEMATC

Commit message: Fabrication outputs
Parts:
- C4: value 1.0uF -> 10uF
- R2: value 1K -> 1k
Changed lines of the file:
@@
 P 5350 9350
 F 0 "R2" V 5154 9350 50  0000 C CNN
-F 1 "1K" V 5245 9350 50  0000 C CNN
+F 1 "1k" V 5245 9350 50  0000 C CNN
 F 2 "Resistor_SMD:R_0805_2012Metric" H 5350 9350 50  0001 C CNN
 F 3 "~" H 5350 9350 50  0001 C CNN
@@
 P 950 9850
 F 0 "C4" H 1042 9896 50  0000 L CNN
-F 1 "1.0uF" H 1042 9805 50  0000 L CNN
+F 1 "10uF" H 1042 9805 50  0000 L CNN
 F 2 "Capacitor_SMD:C_0603_1608Metric" H 950 9850 50  0001 C CNN
 F 3 "~" H 950 9850 50  0001 C CNN
